File: pcb/robot/_autosave-robot.kicad_pcb (KiCad board)
At the start: 2 copper layers, 100 x 100 mm, 5 parts, among them J1 USB_C_Receptacle_USB2.0_16P, Q1 UMH3N, U1 ESP32-WROOM-32, U2 USBLC6-2P6, U3 CP2104

Commit message: added license
Parts:
- added U4: BQ25887, Package_DFN_QFN:VQFN-24-1EP_4x4mm_P0.5mm_EP2.5x2.5mm, F.Cu at (2.65, 2.65)
- moved J1 11.7 mm to (184.0, 57.8)
