File: pcb/robot/_autosave-robot.kicad_sch (KiCad schematic)
At the start: 16 parts, among them J1 USB_C_Receptacle_USB2.0_16P, J2 Conn_01x04_Socket, J3 Conn_01x10_Socket, J4 Conn_01x14_Socket, J5 Conn_01x14_Socket, Q1 UMH3N, U1 ESP32-WROOM-32, U2 USBLC6-2P6, U3 CP2104, U4 BQ25887

Commit message: added license
Parts:
- added J6: Micro_SD_Card_Det1, symbol Connector:Micro_SD_Card_Det1
Changed lines of the file:
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@@
+	)
+	(symbol
+		(lib_id "Connector:Micro_SD_Card_Det1")
+		(at 372.11 91.44 0)
+		(unit 1)
+		(exclude_from_sim no)
+		(in_bom yes)
+		(on_board yes)
+		(dnp no)
+		(fields_autoplaced yes)
+		(property "Reference" "J6"
+			(at 372.745 69.85 0)
+			(effects
+				(font
+					(size 1.27 1.27)
+				)
+			)
+		)
+		(property "Value" "Micro_SD_Card_Det1"
+			(at 372.745 72.39 0)
+			(effects
+				(font
+					(size 1.27 1.27)
+				)
+			)
+		)
+		(property "Footprint" ""
+			(at 424.18 73.66 0)
+			(effects
+				(font
+					(size 1.27 1.27)
+				)
+				(hide yes)
+			)
+		)
+		(property "Datasheet" "https://datasheet.lcsc.com/lcsc/2110151630_XKB-Connectivity-XKTF-015-N_C381082.pdf"
+			(at 372.11 88.9 0)
+			(effects
+				(font
+					(size 1.27 1.27)
+				)
+				(hide yes)
+			)
+		)
+		(property "Description" "Micro SD Card Socket with one card detection pin"
+			(at 372.11 91.44 0)
+			(effects
+				(font
+					(size 1.27 1.27)
+				)
+				(hide yes)
+			)
+		)
+		(pin "8"
+		)
+		(pin "9"
+		)
+		(pin "7"
+		)
+		(pin "1"
+		)
+		(pin "5"
+		)
+		(pin "10"
+		)
+		(pin "3"
+		)
+		(pin "6"
+		)
+		(pin "2"
+		)
+		(pin "4"
+		)
+		(instances
+			(project ""
+				(path "/9447e125-dc0f-40be-afe0-569138d05ba1"
+					(reference "J6")
+					(unit 1)
+				)
+			)
+		)
 	)
 	(symbol
