File: pcb/robot/robot.kicad_pcb (KiCad board)
At the start: 2 copper layers, 5 parts, among them J1 USB_C_Receptacle_USB2.0_16P, Q1 UMH3N, U1 ESP32-WROOM-32, U2 USBLC6-2P6, U3 CP2104

Commit message: Added "Práce_Obsidian"
Parts:
- added J6: Micro_SD_Card_Det1, Connector_Card:microSIM_JAE_SF53S006VCBR2000, F.Cu at (63.5, 65.0)
- added U4: BQ25887, Package_DFN_QFN:VQFN-24-1EP_4x4mm_P0.5mm_EP2.5x2.5mm, F.Cu at (2.65, 2.65)
- added U5: MPU-9250, Sensor_Motion:InvenSense_QFN-24_3x3mm_P0.4mm, F.Cu at (69.9, 90.4)
- added U6: VL53L0CXV0DH1, Sensor_Distance:ST_VL53L1x, F.Cu at (57.3, 53.2)
- added U7: VL53L0CXV0DH1, Sensor_Distance:ST_VL53L1x, F.Cu at (142.6, 53.4)
- added U8: VL53L0CXV0DH1, Sensor_Distance:ST_VL53L1x, B.Cu at (137.2, 53.2)
- added U9: VL53L0CXV0DH1, Sensor_Distance:ST_VL53L1x, B.Cu at (64.2, 53.4)
- moved U3 67.5 mm to (117.4, 62.1)
- moved Q1 60.2 mm to (116.5, 70.6)
- moved U2 47.5 mm to (134.7, 64.5), turned to 0 degrees
- moved J1 40.3 mm to (141.2, 63.9), turned to 90 degrees
- moved U1 37.4 mm to (100.0, 65.7)
Connections:
- U2 pad 1: Net-(J1-D--PadA7) -> Net-(U3-D+)
- U2 pad 3: Net-(J1-D+-PadA6) -> Net-(U3-D-)
- U2 pad 4: Net-(U3-D+) -> Net-(J1-D--PadA7)
- U2 pad 6: Net-(U3-D-) -> Net-(J1-D+-PadA6)
Routing:
- net GND: track 24.3 -> 13.2 mm, vias 1 -> 0
- net +5VP: track 6.70 -> 0.00 mm
- net Net-(U3-D-): track 4.59 -> 0.19 mm
- net +5V: track 6.81 -> 3.24 mm
- net Net-(U3-D+): track 5.36 -> 8.81 mm
- net Net-(J1-D--PadA7): track 7.26 -> 4.78 mm
- net Net-(J1-D+-PadA6): track 4.44 -> 4.76 mm, vias 1 -> 0
Other:
- board outline added: 90 x 100 mm
- board text added: "3V3"
- board text added: "EN"
- board text added: "GND"
- board text added: "IO12"
- board text added: "IO14"
- board text added: "IO23"
- board text added: "IO25"
- board text added: "IO26"
- board text added: "IO27"
- board text added: "IO32"
- board text added: "IO33"
- board text added: "IO34"
- board text added: "IO35"
- board text added: "SENSOR_VN"
- board text added: "SENSOR_VP"
