File: pcb/robot/robot.kicad_sch (KiCad schematic)
At the start: 13 parts, among them J1 USB_C_Receptacle_USB2.0_16P, J2 Conn_01x04_Socket, J3 Conn_01x10_Socket, J4 Conn_01x14_Socket, J5 Conn_01x14_Socket, Q1 UMH3N, U1 ESP32-WROOM-32, U2 USBLC6-2P6, U3 CP2104

Commit message: Added "Práce_Obsidian"
Parts:
- added C1: C_10uF, symbol Device:C_Small
- added C2: C_0.1uF, symbol Device:C_Small
- added J10, J9: Conn_01x06_Socket, symbol Connector:Conn_01x06_Socket
- added J6: Micro_SD_Card_Det1, Connector_Card:microSIM_JAE_SF53S006VCBR2000, symbol Connector:Micro_SD_Card_Det1
- added J7: Conn_01x04_Socket, symbol Connector:Conn_01x04_Socket
- added M1, M2: Motor_DC, symbol Motor:Motor_DC
- added U4: BQ25887, Package_DFN_QFN:VQFN-24-1EP_4x4mm_P0.5mm_EP2.5x2.5mm, symbol Battery_Management:BQ25887
- added U5: MPU-9250, Sensor_Motion:InvenSense_QFN-24_3x3mm_P0.4mm, symbol Sensor_Motion:MPU-9250
- added U6, U7, U8, U9: VL53L0CXV0DH1, Sensor_Distance:ST_VL53L1x, symbol Sensor_Distance:VL53L0CXV0DH1
Connections:
- net +3.3V: now also J7.3 (Pin_3)
- net +5V: now also J7.2 (Pin_2)
- net GND: now also J7.4 (Pin_4)
- net at J1.A7 (D-), J1.B7 (D-): now also U2.4 (I/O2); no longer U2.1 (I/O1)
- net at J1.A6 (D+), J1.B6 (D+): now also U2.6 (I/O1); no longer U2.3 (I/O2)
- net at U3.3 (D+): now also U2.1 (I/O1); no longer U2.4 (I/O2)
- net at U3.4 (D-): now also U2.3 (I/O2); no longer U2.6 (I/O1)
- new net: U9.12 (GND), U9.3 (GND), U9.4 (GND), U9.6 (GND)
- new net: U6.12 (GND), U6.3 (GND), U6.4 (GND), U6.6 (GND)
- new net: U8.12 (GND), U8.3 (GND), U8.4 (GND), U8.6 (GND)
- new net: U7.12 (GND), U7.3 (GND), U7.4 (GND), U7.6 (GND)
- new net: U4.13 (BAT), U4.14 (BAT)
- new net: U4.15 (SNS), U4.16 (SNS)
- new net: U4.17 (SW), U4.18 (SW)
- new net: U4.19 (GND), U4.20 (GND)
- new net: U4.21 (PMID), U4.22 (PMID)
- new net +12V: J7.1 (Pin_1)
- no-connect marks 0 -> 4
Other:
- added sheet PSU (untitled.kicad_sch)
- moved on the sheet: U2

Commit message: 30.1.2025 no big changes, going to get latex runing
Parts:
- added BMS1: 2S 20A, symbol personalized_symbols:HW-391
- added Charger1: ~, symbol personalized_symbols:TP5100
- added Q2, Q3, Q4: NMOS, symbol Simulation_SPICE:NMOS
- added R3: 68k, symbol Device:R
- added R4: 33k, symbol Device:R
- added STP_DOWN1: ~, symbol personalized_symbols:Step_down
- added STP_UP1, STP_UP2: ~, symbol personalized_symbols:Step_Up
- added ncr18650ga1, ncr18650ga2: 2.5-4.2V, symbol Device:Battery_Cell
Connections:
- net GND: now also BMS1.5 (OUT_GND), Charger1. (OUT_GND), R4.2, STP_DOWN1. (VOUT), STP_UP1. (VOUT), STP_UP2. (VOUT)
- new net: BMS1.1 (8.4V), ncr18650ga1.1 (+)
- new net: BMS1.2 (4.2V), ncr18650ga1.2 (-), ncr18650ga2.1 (+)
- new net: Q2.3 (S), STP_DOWN1. (VOUT), STP_UP1. (VOUT)
- new net: Q3.3 (S), STP_UP2. (VOUT)
- new net: BMS1.4 (OUT_8.4V), Charger1. (OUT_GND), Q2.1 (D), Q3.1 (D), Q4.1 (D)
- new net: BMS1.3 (0V), ncr18650ga2.2 (-)
- new net: Q4.3 (S), R3.1
- new net 3.3V: STP_DOWN1. (VOUT)
- new net Bridge1_12V: STP_UP1. (VOUT)
- new net Bridge2_12V: STP_UP2. (VOUT)
- new net Bridge2_GND: STP_UP2. (VOUT)
- new net Brigde1_GND: STP_UP1. (VOUT)
- new net Charging_5-15V: Charger1. (OUT_GND)
- new net Charging_GND: Charger1. (OUT_GND)
- new net activate_motors: Q2.2 (G), Q3.2 (G)
- new net activate_voltage_divider: Q4.2 (G)
- new net measure_voltage_high: R3.2, R4.1
