File: pcb/1_robot/esp32.kicad_sch (KiCad schematic)
At the start: 1 part, among them U1 ESP32-WROOM-32D

Commit message: finished work
Parts:
- removed U1: ESP32-WROOM-32D, RF_Module:ESP32-WROOM-32D, symbol RF_Module:ESP32-WROOM-32D
- added C14, C5: 12u, symbol Device:C
- added C6, C7: 0.1u, symbol Device:C
- added C8: 22u, symbol Device:C
- added C9: C, symbol Device:C
- added J11: Conn_01x10_Pin, Connector_PinHeader_2.54mm:PinHeader_2x05_P2.54mm_Vertical, symbol Connector:Conn_01x10_Pin
- added J6: Micro_SD_Card_Det1, Connector_Card:microSD_HC_Wuerth_693072010801, symbol Connector:Micro_SD_Card_Det1
- added J7, J9: Conn_01x14_Pin, Connector_PinHeader_2.54mm:PinHeader_2x07_P2.54mm_Vertical, symbol Connector:Conn_01x14_Pin
- added R2: 10k, symbol Device:R
- added R3: R, symbol Device:R
- added SW1, SW2: SW_Push, symbol Switch:SW_Push
- added U3: ESP32-WROOM-32E, RF_Module:ESP32-WROOM-32D, symbol RF_Module:ESP32-WROOM-32E
- added Y3: Crystal, Oscillator:Oscillator_SMD_Abracon_ASCO-4Pin_1.6x1.2mm, symbol Device:Crystal
Connections:
- new net 3V3: C7.2, C8.2, J6.4 (VDD), J7.2 (Pin_2), R2.2, R3.2, U3.2 (VDD)
- new net Activate_Motors: J9.13 (Pin_13), U3.26 (IO4)
- new net CLK: J11.6 (Pin_6)
- new net CMD: J11.5 (Pin_5)
- new net CS_1: J6.2 (DAT3/CD), J9.10 (Pin_10), U3.29 (IO5)
- new net EN: C6.2, J7.3 (Pin_3), R2.1, SW1.2, U3.3 (EN)
- new net Feedback_1_1: J7.10 (Pin_10), U3.10 (IO25)
- new net Feedback_1_2: J7.11 (Pin_11), U3.11 (IO26)
- new net Feedback_2_1: J7.12 (Pin_12), U3.12 (IO27)
- new net Feedback_2_2: J7.6 (Pin_6), U3.6 (IO34)
- new net GND: C14.2, C5.2, C6.1, C7.1, C8.1, C9.1, J11.1 (Pin_1), J6.6 (VSS), J7.1 (Pin_1), J9.1 (Pin_1), SW1.1, SW2.1, U3.1 (GND), U3.15 (GND), U3.38 (GND), U3.39 (GND)
- new net IO0: C9.2, J9.14 (Pin_14), R3.1, SW2.2, U3.25 (IO0)
- new net IO17: J9.11 (Pin_11), U3.28 (IO17)
- new net IO18: J6.5 (CLK), J9.9 (Pin_9), U3.30 (IO18)
- new net IO19: J6.7 (DAT0), J9.8 (Pin_8), U3.31 (IO19)
- new net IO2: J11.10 (Pin_10), U3.24 (IO2)
- new net IO21: J9.6 (Pin_6), U3.33 (IO21)
- new net IO22: J9.3 (Pin_3), U3.36 (IO22)
- new net IO23: J6.3 (CMD), J9.2 (Pin_2), U3.37 (IO23)
- new net IO32: C14.1, J7.8 (Pin_8), U3.8 (IO32), Y3.2
- new net IO33: C5.1, J7.9 (Pin_9), U3.9 (IO33), Y3.1
- new net M_1_A: J7.14 (Pin_14), U3.14 (IO12)
- new net M_1_B: J11.2 (Pin_2), U3.16 (IO13)
- new net M_2_A: J7.13 (Pin_13), U3.13 (IO14)
- new net M_2_B: J11.9 (Pin_9), U3.23 (IO15)
- new net Measure_Voltage: J7.7 (Pin_7), U3.7 (IO35)
- new net NC: J9.7 (Pin_7)
- new net NeoPixel: J9.12 (Pin_12), U3.27 (IO16)
- new net RX_PRG: J9.5 (Pin_5), U3.34 (RXD0/IO3)
- new net SD0: J11.7 (Pin_7)
- new net SD1: J11.8 (Pin_8)
- new net SD2: J11.3 (Pin_3)
- new net SD3: J11.4 (Pin_4)
- new net Sensor_VN: J7.5 (Pin_5), U3.5 (SENSOR_VN)
- new net Sensor_VP: J7.4 (Pin_4), U3.4 (SENSOR_VP)
- new net TX_PRG: J9.4 (Pin_4), U3.35 (TXD0/IO1)
- no-connect marks 0 -> 21
Other:
- note added: "ESP S3"
- note added: "https://randomnerdtutorials.com/esp32-i2c-communication-arduino-ide/"
- note added: "https://randomnerdtutorials.com/esp32-microsd-card-arduino/"
- note added: "https://randomnerdtutorials.com/esp32-pinout-reference-gpios/"
- note added: "https://randomnerdtutorials.com/esp32-spi-communication-arduino/"
- note added: "https://www.youtube.com/watch?v=S_p0YV-JlfU"
