File: pcb/1_robot/input.kicad_sch (KiCad schematic)
At the start: 1 part, among them P1 USB_C_Plug_USB2.0

Commit message: finished work
Parts:
- removed P1: USB_C_Plug_USB2.0, symbol Connector:USB_C_Plug_USB2.0
- added C11: C, Capacitor_SMD:C_0603_1608Metric_Pad1.08x0.95mm_HandSolder, symbol Device:C
- added C12, C13, C4: C, Capacitor_SMD:C_0402_1005Metric_Pad0.74x0.62mm_HandSolder, symbol Device:C
- added C19: 10u, symbol Device:C
- added C20, C22: 1u, symbol Device:C
- added C21, C3: 100n, symbol Device:C
- added D4, D5: LED, symbol Device:LED
- added J5: USB_C_Receptacle_USB2.0_16P, Connector_USB:USB_C_Receptacle_HCTL_HC-TYPE-C-16P-01A, symbol Connector:USB_C_Receptacle_USB2.0_16P
- added Q7, Q8: NMOS, symbol Simulation_SPICE:NMOS
- added R10, R7, R9: 100k, symbol Device:R
- added R11, R14, R15, R20, R24, R25, R26, R27: 0, symbol Device:R
- added R12, R13: 5k1, symbol Device:R
- added R16: 27k, symbol Device:R
- added R17, R21: 10k, symbol Device:R
- added R18: 10m, symbol Device:R
- added R19: 100, symbol Device:R
- added U4: CH340G, Package_SO:SOIC-16_3.9x9.9mm_P1.27mm, symbol Interface_USB:CH340G
- added U5: AP33771DKZ-13, AP33771DKZ-13:IC_AP33771DKZ-13, symbol personalized_symbols:AP33771DKZ-13
- added Y2: Crystal_GND24, Oscillator:Oscillator_SMD_Abracon_ASE-4Pin_3.2x2.5mm_HandSoldering, symbol Device:Crystal_GND24
Connections:
- new net: R16.1, U5.13 (PSEL)
- new net: D4.2 (A), R17.2
- new net: Q7.2 (G), Q8.2 (G), R19.2
- new net: Q7.3 (S), Q8.3 (S)
- new net: C13.1, U4.8 (XO), Y2.3
- new net: U5.10 (NC), U5.18 (NC), U5.19 (NC), U5.2 (NC), U5.21 (NC), U5.4 (NC), U5.5 (NC)
- new net: C21.1, U5.12 (V3VD)
- new net: C3.1, U5.15 (IFB)
- new net: C22.1, U5.20 (V5V)
- new net: R21.1, U5.6 (GPIO4)
- new net: R24.1, U4.2 (TXD)
- new net: R25.1, U4.3 (RXD)
- new net: R26.2, U4.5 (UD+)
- new net: R27.2, U4.6 (UD-)
- new net: C4.1, U4.7 (XI), Y2.1
- new net: D5.2 (A), R21.2
- new net 3V3: C11.1, C12.1, R11.1, R14.1, R15.1, U4.16 (VCC), U4.4 (V3)
- new net CC1: J5.A5 (CC1), R12.1, U5.17 (CC1)
- new net CC2: J5.B5 (CC2), R13.1, U5.16 (CC2)
- new net D+: J5.A6 (D+), J5.B6 (D+), R26.1
- new net D-: J5.A7 (D-), J5.B7 (D-), R27.1
- new net GND: C11.2, C12.2, C13.2, C19.2, C20.2, C21.2, C22.2, C3.2, C4.2, D4.1 (K), D5.1 (K), J5.A1 (GND), J5.A12 (GND), J5.B1 (GND), J5.B12 (GND), J5.S1 (SHIELD), R10.2, R12.2, R13.2, R16.2, R7.2, R9.2, U4.1 (GND), U5.3 (GND), Y2.2, Y2.4
- new net PD_VOUT: C20.1, Q8.1 (D), R20.1
- new net PWR_EN: R19.1, U5.23 (PWR_EN)
- new net RX: R25.2
- new net TX: R24.2
- new net VBUS: R20.2, U5.22 (VBUS)
- new net VBUS_USB: C19.1, J5.A4 (VBUS), J5.A9 (VBUS), J5.B4 (VBUS), J5.B9 (VBUS), R17.1, R18.1, U5.1 (ISENP)
- new net VCC: Q7.1 (D), R18.2, U5.24 (VCC)
- new net VSEL0: R11.2, R7.1, U5.9 (VSEL0)
- new net VSEL1: R14.2, R9.1, U5.7 (VSEL1)
- new net VSEL2: R10.1, R15.2, U5.11 (VSEL2)
- no-connect marks 0 -> 12
Other:
- note added: "Power Delivery"
- note added: "USB to UART"
- note added: "https://components101.com/misc/microsd-card-pinout-datasheet"
- note added: "https://randomnerdtutorials.com/esp32-microsd-card-arduino/"
- note added: "https://static.efetividade.net/img/ch340g-datasheet-34852.pdf"
- note added: "protection"
- note added: "usb to UART"
